Commit message: changes required for realsense camera affixed to the bracelet cuff

File: kortex_description/arms/gen3/7dof/urdf/gen3_macro.xacro (robot description, xacro)
@@ -312,4 +312,14 @@
     <xacro:if value="${vision}">
       <link name="${prefix}camera_link" />
+      <gazebo>
+        <include>
+          <uri>model://realsense_camera</uri>
+          <pose>-0.045 0.04 1.185 1.57 -1.57 0</pose>
+        </include>
+        <joint name="camera_joint" type="fixed">
+          <child>realsense_camera::link</child>
+          <parent>camera_link</parent>
+        </joint>
+      </gazebo>
       <joint name="${prefix}camera_module" type="fixed">
         <origin xyz="0 0.05639 -0.00305" rpy="3.14159265358979 3.14159265358979 0" />

Commit message: setup with fixed camera complete

File: kortex_description/arms/gen3/7dof/urdf/gen3_macro.xacro (robot description, xacro)
@@ -312,14 +312,4 @@
     <xacro:if value="${vision}">
       <link name="${prefix}camera_link" />
-      <gazebo>
-        <include>
-          <uri>model://realsense_camera</uri>
-          <pose>-0.045 0.04 1.185 1.57 -1.57 0</pose>
-        </include>
-        <joint name="camera_joint" type="fixed">
-          <child>realsense_camera::link</child>
-          <parent>camera_link</parent>
-        </joint>
-      </gazebo>
       <joint name="${prefix}camera_module" type="fixed">
         <origin xyz="0 0.05639 -0.00305" rpy="3.14159265358979 3.14159265358979 0" />
@@ -340,4 +330,10 @@
       </joint>
     </xacro:if>
+      <gazebo>
+        <include>
+          <uri>model://realsense_camera</uri>
+          <pose>0.8 0.0 .8 1.57 1.57 1.57</pose>
+        </include>
+      </gazebo>
   </xacro:macro>
 </robot>

Commit message: added fixed camera to this branch

File: kortex_description/arms/gen3/7dof/urdf/gen3_macro.xacro (robot description, xacro)
@@ -312,14 +312,4 @@
     <xacro:if value="${vision}">
       <link name="${prefix}camera_link" />
-      <gazebo>
-        <include>
-          <uri>model://realsense_camera</uri>
-          <pose>0.045 0.04 1.185 -1.57 -1.57 0</pose>
-        </include>
-        <joint name="camera_joint" type="fixed">
-          <child>realsense_camera::link</child>
-          <parent>camera_link</parent>
-        </joint>
-      </gazebo>
       <joint name="${prefix}camera_module" type="fixed">
         <origin xyz="0 0.05639 -0.00305" rpy="3.14159265358979 3.14159265358979 0" />
@@ -340,4 +330,10 @@
       </joint>
     </xacro:if>
+      <gazebo>
+        <include>
+          <uri>model://realsense_camera</uri>
+          <pose>0.5 -0.2 0.55 -1.57 1.70 1.57</pose>
+        </include>
+      </gazebo>
   </xacro:macro>
 </robot>

Commit message: Fixed camera issue

File: kortex_description/arms/gen3/7dof/urdf/gen3_macro.xacro (robot description, xacro)
@@ -311,15 +311,9 @@
     </joint>
     <xacro:if value="${vision}">
-      <link name="${prefix}camera_link" />
-      <gazebo>
-        <include>
-          <uri>model://realsense_camera</uri>
-          <pose>0.045 0.04 1.185 -1.57 -1.57 0</pose>
-        </include>
-        <joint name="camera_joint" type="fixed">
-          <child>realsense_camera::link</child>
-          <parent>camera_link</parent>
-        </joint>
-      </gazebo>
+			<link name="${prefix}camera_link"/>
+			<xacro:include filename="$(find realsense_gazebo_plugin)/urdf/realsense-RS200.macro.xacro"/>
+	    <xacro:realsense-rs200 prefix="${prefix}" parent="camera_link">
+				<origin xyz="0.0 0.0 0.01" rpy="0 -1.57 1.57" />
+	    </xacro:realsense-rs200>
       <joint name="${prefix}camera_module" type="fixed">
         <origin xyz="0 0.05639 -0.00305" rpy="3.14159265358979 3.14159265358979 0" />
